File: Attiny85_ProgBoard_v1.kicad_pcb (KiCad board)
At the start: 2 copper layers, 1 part, among them U1 ATtiny85V-10PU

Commit message: worked on PCB design
Parts:
- moved U1 12.8 mm to (139.7, 86.4)
Connections:
- U1 pad 1: Net-(U1-Pad1) -> unconnected-(U1-~{RESET}/PB5-Pad1)
- U1 pad 2: Net-(U1-Pad2) -> unconnected-(U1-XTAL1/PB3-Pad2)
- U1 pad 3: Net-(U1-Pad3) -> unconnected-(U1-XTAL2/PB4-Pad3)
- U1 pad 4: Net-(U1-Pad4) -> unconnected-(U1-GND-Pad4)
- U1 pad 5: Net-(U1-Pad5) -> unconnected-(U1-AREF/PB0-Pad5)
- U1 pad 6: Net-(U1-Pad6) -> unconnected-(U1-PB1-Pad6)
- U1 pad 7: Net-(U1-Pad7) -> unconnected-(U1-PB2-Pad7)
- U1 pad 8: Net-(U1-Pad8) -> unconnected-(U1-VCC-Pad8)
Other:
- board outline added: 22.9 x 22.9 mm
- net class Default removed

Commit message: Designed PCB
Parts:
- added AREF/PB0: Conn_01x01_Female, Connector_Pin:PinHole_01x01, F.Cu at (162.6, 94.0)
- added GND: Conn_01x01_Female, Connector_Pin:PinHole_01x01, F.Cu at (124.5, 94.0)
- added PB1: Conn_01x01_Female, Connector_Pin:PinHole_01x01, F.Cu at (162.6, 91.4)
- added PB2: Conn_01x01_Female, Connector_Pin:PinHole_01x01, F.Cu at (162.6, 88.9)
- added VCC: Conn_01x01_Female, Connector_Pin:PinHole_01x01, F.Cu at (162.6, 86.4)
- added XTAL1/PB3: Conn_01x01_Female, Connector_Pin:PinHole_01x01, F.Cu at (124.5, 88.9)
- added XTAL2/PB4: Conn_01x01_Female, Connector_Pin:PinHole_01x01, F.Cu at (124.5, 91.4)
- added ~{RESET}/PB5: Conn_01x01_Female, Connector_Pin:PinHole_01x01, F.Cu at (124.5, 86.4)
- renumbered U1 to ATTINY85
Connections:
- ATTINY85 pad 1: unconnected-(U1-~{RESET}/PB5-Pad1) -> Net-(J7-Pin_1)
- ATTINY85 pad 2: unconnected-(U1-XTAL1/PB3-Pad2) -> Net-(J5-Pin_1)
- ATTINY85 pad 3: unconnected-(U1-XTAL2/PB4-Pad3) -> Net-(J6-Pin_1)
- ATTINY85 pad 4: unconnected-(U1-GND-Pad4) -> Net-(J8-Pin_1)
- ATTINY85 pad 5: unconnected-(U1-AREF/PB0-Pad5) -> Net-(J2-Pin_1)
- ATTINY85 pad 6: unconnected-(U1-PB1-Pad6) -> Net-(J3-Pin_1)
- ATTINY85 pad 7: unconnected-(U1-PB2-Pad7) -> Net-(J4-Pin_1)
- ATTINY85 pad 8: unconnected-(U1-VCC-Pad8) -> Net-(J1-Pin_1)
Routing:
- net Net-(J4-Pin_1): track 0.00 -> 15.2 mm
- net Net-(J3-Pin_1): track 0.00 -> 15.2 mm
- net Net-(J2-Pin_1): track 0.00 -> 15.2 mm
- net Net-(J1-Pin_1): track 0.00 -> 15.2 mm
- net Net-(J8-Pin_1): track 0.00 -> 15.2 mm
- net Net-(J7-Pin_1): track 0.00 -> 15.2 mm
- net Net-(J6-Pin_1): track 0.00 -> 15.2 mm
- net Net-(J5-Pin_1): track 0.00 -> 15.2 mm
Other:
- board size 22.9 x 22.9 mm -> 43.2 x 17.8 mm

Commit message: Added GND planes on top layer
Parts:
- renumbered GND to GND1, ATTINY85 to U1, VCC to VCC1, ~{RESET}/PB5 to ~RESET/PB4
Connections:
- AREF/PB0 pad 1: Net-(J2-Pin_1) -> (no net)
- GND1 pad 1: Net-(J8-Pin_1) -> (no net)
- PB1 pad 1: Net-(J3-Pin_1) -> (no net)
- PB2 pad 1: Net-(J4-Pin_1) -> (no net)
- U1 pad 4: Net-(J8-Pin_1) -> Net-(GND1-Pin_1)
- U1 pad 5: Net-(J2-Pin_1) -> Net-(AREF/PB0-Pin_1)
- U1 pad 6: Net-(J3-Pin_1) -> Net-(PB1-Pin_1)
- U1 pad 7: Net-(J4-Pin_1) -> Net-(PB2-Pin_1)
Routing:
- net Net-(PB2-Pin_1): track 0.00 -> 15.2 mm
- net Net-(PB1-Pin_1): track 0.00 -> 15.2 mm
- net Net-(J4-Pin_1): track 15.2 -> 0.00 mm
- net Net-(J3-Pin_1): track 15.2 -> 0.00 mm
- net Net-(J2-Pin_1): track 15.2 -> 0.00 mm
- net Net-(AREF/PB0-Pin_1): track 0.00 -> 15.2 mm
- net Net-(J8-Pin_1): track 15.2 -> 0.00 mm
- added copper zone on F.Cu, net Net-(GND1-Pin_1)
Changed lines of the file:
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@@
   )
   (net 0 "")
-  (net 1 "Net-(J1-Pin_1)")
-  (net 2 "Net-(J2-Pin_1)")
-  (net 3 "Net-(J8-Pin_1)")
-  (net 4 "Net-(J7-Pin_1)")
-  (net 5 "Net-(J6-Pin_1)")
-  (net 6 "Net-(J5-Pin_1)")
-  (net 7 "Net-(J4-Pin_1)")
-  (net 8 "Net-(J3-Pin_1)")
+  (net 1 "Net-(AREF/PB0-Pin_1)")
+  (net 2 "Net-(GND1-Pin_1)")
+  (net 3 "Net-(PB1-Pin_1)")
+  (net 4 "Net-(PB2-Pin_1)")
+  (net 5 "Net-(U1-~{RESET}{slash}PB5)")
+  (net 6 "Net-(U1-XTAL1{slash}PB3)")
+  (net 7 "Net-(U1-XTAL2{slash}PB4)")
+  (net 8 "Net-(U1-VCC)")
   (footprint "Connector_Pin:PinHole_01x01" (layer "F.Cu")
     (at 124.46 88.9)
@@
     )
     (pad "1" thru_hole circle (at 0 0) (size 1.524 1.524) (drill 0.762) (layers "*.Cu" "*.Mask")
-      (net 6 "Net-(J5-Pin_1)") (pinfunction "Pin_1") (pintype "passive"))
+      (net 6 "Net-(U1-XTAL1{slash}PB3)") (pinfunction "Pin_1") (pintype "passive"))
   )
   (footprint "Connector_Pin:PinHole_01x01" (layer "F.Cu")
@@
     (property "ki_keywords" "connector")
     (attr through_hole)
-    (fp_text reference "VCC" (at -3.175 -1.0414 unlocked) (layer "F.SilkS")
-        (effects (font (size 1 1) (thickness 0.1)))
-    )
-    (fp_text value "Conn_01x01_Female" (at 0 -2.54 unlocked) (layer "F.Fab")
-        (effects (font (size 1 1) (thickness 0.15)))
-    )
-    (fp_text user "${REFERENCE}" (at 0.075 2.475 unlocked) (layer "F.Fab")
-        (effects (font (size 1 1) (thickness 0.15)))
-    )
-    (pad "1" thru_hole circle (at 0 0) (size 1.524 1.524) (drill 0.762) (layers "*.Cu" "*.Mask")
-      (net 1 "Net-(J1-Pin_1)") (pinfunction "Pin_1") (pintype "passive"))
+    (fp_text reference "VCC1" (at -3.175 -1.0414 unlocked) (layer "F.SilkS")
+        (effects (font (size 1 1) (thickness 0.1)))
+    )
+    (fp_text value "Conn_01x01_Female" (at 0 -2.54 unlocked) (layer "F.Fab")
+        (effects (font (size 1 1) (thickness 0.15)))
+    )
+    (fp_text user "${REFERENCE}" (at 0.075 2.475 unlocked) (layer "F.Fab")
+        (effects (font (size 1 1) (thickness 0.15)))
+    )
+    (pad "1" thru_hole circle (at 0 0) (size 1.524 1.524) (drill 0.762) (layers "*.Cu" "*.Mask")
+      (net 8 "Net-(U1-VCC)") (pinfunction "Pin_1") (pintype "passive"))
   )
   (footprint "Connector_Pin:PinHole_01x01" (layer "F.Cu")
@@
     )
     (pad "1" thru_hole circle (at 0 0) (size 1.524 1.524) (drill 0.762) (layers "*.Cu" "*.Mask")
-      (net 5 "Net-(J6-Pin_1)") (pinfunction "Pin_1") (pintype "passive"))
+      (net 7 "Net-(U1-XTAL2{slash}PB4)") (pinfunction "Pin_1") (pintype "passive"))
   )
   (footprint "Package_DIP:DIP-8_W7.62mm" (layer "F.Cu")
@@
     (property "Sheetname" "")
     (attr through_hole)
-    (fp_text reference "ATTINY85" (at 3.81 -2.33) (layer "F.SilkS")
+    (fp_text reference "U1" (at 3.81 -2.33) (layer "F.SilkS")
         (effects (font (size 1 1) (thickness 0.15)))
     )
@@
       (stroke (width 0.1) (type solid)) (layer "F.Fab"))
     (pad "1" thru_hole rect (at 0 0) (size 1.6 1.6) (drill 0.8) (layers "*.Cu" "*.Mask")
-      (net 4 "Net-(J7-Pin_1)") (pinfunction "~{RESET}/PB5") (pintype "bidirectional"))
+      (net 5 "Net-(U1-~{RESET}{slash}PB5)") (pinfunction "~{RESET}/PB5") (pintype "bidirectional"))
     (pad "2" thru_hole oval (at 0 2.54) (size 1.6 1.6) (drill 0.8) (layers "*.Cu" "*.Mask")
-      (net 6 "Net-(J5-Pin_1)") (pinfunction "XTAL1/PB3") (pintype "bidirectional"))
+      (net 6 "Net-(U1-XTAL1{slash}PB3)") (pinfunction "XTAL1/PB3") (pintype "bidirectional"))
     (pad "3" thru_hole oval (at 0 5.08) (size 1.6 1.6) (drill 0.8) (layers "*.Cu" "*.Mask")
-      (net 5 "Net-(J6-Pin_1)") (pinfunction "XTAL2/PB4") (pintype "bidirectional"))
+      (net 7 "Net-(U1-XTAL2{slash}PB4)") (pinfunction "XTAL2/PB4") (pintype "bidirectional"))
     (pad "4" thru_hole oval (at 0 7.62) (size 1.6 1.6) (drill 0.8) (layers "*.Cu" "*.Mask")
-      (net 3 "Net-(J8-Pin_1)") (pinfunction "GND") (pintype "power_in"))
+      (net 2 "Net-(GND1-Pin_1)") (pinfunction "GND") (pintype "power_in"))
     (pad "5" thru_hole oval (at 7.62 7.62) (size 1.6 1.6) (drill 0.8) (layers "*.Cu" "*.Mask")
-      (net 2 "Net-(J2-Pin_1)") (pinfunction "AREF/PB0") (pintype "bidirectional"))
+      (net 1 "Net-(AREF/PB0-Pin_1)") (pinfunction "AREF/PB0") (pintype "bidirectional"))
     (pad "6" thru_hole oval (at 7.62 5.08) (size 1.6 1.6) (drill 0.8) (layers "*.Cu" "*.Mask")
-      (net 8 "Net-(J3-Pin_1)") (pinfunction "PB1") (pintype "bidirectional"))
+      (net 3 "Net-(PB1-Pin_1)") (pinfunction "PB1") (pintype "bidirectional"))
     (pad "7" thru_hole oval (at 7.62 2.54) (size 1.6 1.6) (drill 0.8) (layers "*.Cu" "*.Mask")
-      (net 7 "Net-(J4-Pin_1)") (pinfunction "PB2") (pintype "bidirectional"))
+      (net 4 "Net-(PB2-Pin_1)") (pinfunction "PB2") (pintype "bidirectional"))
     (pad "8" thru_hole oval (at 7.62 0) (size 1.6 1.6) (drill 0.8) (layers "*.Cu" "*.Mask")
-      (net 1 "Net-(J1-Pin_1)") (pinfunction "VCC") (pintype "power_in"))
+      (net 8 "Net-(U1-VCC)") (pinfunction "VCC") (pintype "power_in"))
     (model "${KICAD6_3DMODEL_DIR}/Package_DIP.3dshapes/DIP-8_W7.62mm.wrl"
       (offset (xyz 0 0 0))
@@
     )
     (pad "1" thru_hole circle (at 0 0) (size 1.524 1.524) (drill 0.762) (layers "*.Cu" "*.Mask")
-      (net 2 "Net-(J2-Pin_1)") (pinfunction "Pin_1") (pintype "passive"))
+      (pinfunction "Pin_1") (pintype "passive"))
   )
   (footprint "Connector_Pin:PinHole_01x01" (layer "F.Cu")
@@
     )
     (pad "1" thru_hole circle (at 0 0) (size 1.524 1.524) (drill 0.762) (layers "*.Cu" "*.Mask")
-      (net 8 "Net-(J3-Pin_1)") (pinfunction "Pin_1") (pintype "passive"))
+      (pinfunction "Pin_1") (pintype "passive"))
   )
   (footprint "Connector_Pin:PinHole_01x01" (layer "F.Cu")
@@
     )
     (pad "1" thru_hole circle (at 0 0) (size 1.524 1.524) (drill 0.762) (layers "*.Cu" "*.Mask")
-      (net 7 "Net-(J4-Pin_1)") (pinfunction "Pin_1") (pintype "passive"))
+      (pinfunction "Pin_1") (pintype "passive"))
   )
   (footprint "Connector_Pin:PinHole_01x01" (layer "F.Cu")
@@
     (property "ki_keywords" "connector")
     (attr through_hole)
-    (fp_text reference "GND" (at 2.7178 -0.8128 unlocked) (layer "F.SilkS")
-        (effects (font (size 1 1) (thickness 0.1)))
-    )
-    (fp_text value "Conn_01x01_Female" (at 0 -2.54 unlocked) (layer "F.Fab")
-        (effects (font (size 1 1) (thickness 0.15)))
-    )
-    (fp_text user "${REFERENCE}" (at 0.075 2.475 unlocked) (layer "F.Fab")
-        (effects (font (size 1 1) (thickness 0.15)))
-    )
-    (pad "1" thru_hole circle (at 0 0) (size 1.524 1.524) (drill 0.762) (layers "*.Cu" "*.Mask")
-      (net 3 "Net-(J8-Pin_1)") (pinfunction "Pin_1") (pintype "passive"))
+    (fp_text reference "GND1" (at 2.7178 -0.8128 unlocked) (layer "F.SilkS")
+        (effects (font (size 1 1) (thickness 0.1)))
+    )
+    (fp_text value "Conn_01x01_Female" (at 0 -2.54 unlocked) (layer "F.Fab")
+        (effects (font (size 1 1) (thickness 0.15)))
+    )
+    (fp_text user "${REFERENCE}" (at 0.075 2.475 unlocked) (layer "F.Fab")
+        (effects (font (size 1 1) (thickness 0.15)))
+    )
+    (pad "1" thru_hole circle (at 0 0) (size 1.524 1.524) (drill 0.762) (layers "*.Cu" "*.Mask")
+      (pinfunction "Pin_1") (pintype "passive"))
   )
   (footprint "Connector_Pin:PinHole_01x01" (layer "F.Cu")
@@
     (property "ki_keywords" "connector")
     (attr through_hole)
-    (fp_text reference "~{RESET}/PB5" (at 1.143 -1.0414 unlocked) (layer "F.SilkS")
+    (fp_text reference "~RESET/PB4" (at 1.143 -1.0414 unlocked) (layer "F.SilkS")
         (effects (font (size 1 1) (thickness 0.1)) (justify left))
     )
@@
     )
     (pad "1" thru_hole circle (at 0 0) (size 1.524 1.524) (drill 0.762) (layers "*.Cu" "*.Mask")
-      (net 4 "Net-(J7-Pin_1)") (pinfunction "Pin_1") (pintype "passive"))
+      (net 5 "Net-(U1-~{RESET}{slash}PB5)") (pinfunction "Pin_1") (pintype "passive"))
   )
   (gr_rect (start 121.92 81.28) (end 165.1 99.06)
     (stroke (width 0.1) (type default)) (fill none) (layer "Edge.Cuts"))
-  (segment (start 147.32 86.36) (end 162.56 86.36) (width 0.25) (layer "F.Cu") (net 1))
-  (segment (start 162.56 93.98) (end 147.32 93.98) (width 0.25) (layer "F.Cu") (net 2))
-  (segment (start 124.46 93.98) (end 139.7 93.98) (width 0.25) (layer "F.Cu") (net 3))
-  (segment (start 124.46 86.36) (end 139.7 86.36) (width 0.25) (layer "F.Cu") (net 4))
-  (segment (start 124.46 91.44) (end 139.7 91.44) (width 0.25) (layer "F.Cu") (net 5))
+  (segment (start 162.56 93.98) (end 147.32 93.98) (width 0.25) (layer "F.Cu") (net 1))
+  (segment (start 147.32 91.44) (end 162.56 91.44) (width 0.25) (layer "F.Cu") (net 3))
+  (segment (start 147.32 88.9) (end 162.56 88.9) (width 0.25) (layer "F.Cu") (net 4))
+  (segment (start 124.46 86.36) (end 139.7 86.36) (width 0.25) (layer "F.Cu") (net 5))
   (segment (start 124.46 88.9) (end 139.7 88.9) (width 0.25) (layer "F.Cu") (net 6))
-  (segment (start 147.32 88.9) (end 162.56 88.9) (width 0.25) (layer "F.Cu") (net 7))
-  (segment (start 147.32 91.44) (end 162.56 91.44) (width 0.25) (layer "F.Cu") (net 8))
+  (segment (start 124.46 91.44) (end 139.7 91.44) (width 0.25) (layer "F.Cu") (net 7))
+  (segment (start 147.32 86.36) (end 162.56 86.36) (width 0.25) (layer "F.Cu") (net 8))
+  (zone (net 2) (net_name "Net-(GND1-Pin_1)") (layer "F.Cu") (hatch edge 0.5)
+    (connect_pads (clearance 0.508))
+    (min_thickness 0.25) (filled_areas_thickness no)
+    (fill yes (thermal_gap 0.5) (thermal_bridge_width 0.5))
+    (polygon
+      (pts
+        (xy 121.92 81.28)
+        (xy 165.1 81.28)
+        (xy 165.1 99.06)
+        (xy 121.92 99.06)
+      )
+    )
+  )
 )

Commit message: Added dedicated library
Parts:
- removed GND1, VCC1, ~RESET/PB4: Conn_01x01_Female, Connector_Pin:PinHole_01x01
- added GND: Conn_01x01_Female, PinHole:PinHole_01x01, F.Cu at (124.5, 94.0)
- added VCC: Conn_01x01_Female, PinHole:PinHole_01x01, F.Cu at (162.3, 86.4)
- added ~{RESET}/PB5: Conn_01x01_Female, PinHole:PinHole_01x01, F.Cu at (124.5, 86.4)
- AREF/PB0, PB1, PB2, XTAL1/PB3, XTAL2/PB4: footprint Connector_Pin:PinHole_01x01 -> PinHole:PinHole_01x01
- moved PB1 0.25 mm to (162.3, 91.4)
- moved PB2 0.25 mm to (162.3, 88.9)
- renumbered U1 to ATTINY85
Connections:
- AREF/PB0 pad 1: (no net) -> Net-(AREF/PB0-Pin_1)
- PB1 pad 1: (no net) -> Net-(PB1-Pin_1)
- PB2 pad 1: (no net) -> Net-(PB2-Pin_1)
